Commit message: iarrc pointcloud conversion and planning

File: rr_description/urdf/sedani.urdf (robot description, URDF)
Before this commit: robot macaroni, 22 links, 21 joints
Joints:
- joint camera_joint: origin xyz=0.28 0 0.267 rpy=0 0 0 -> xyz=0.28 0 0.267 rpy=0 0.02 0

Commit message: image_transform improvements

File: rr_description/urdf/sedani.urdf (robot description, URDF)
Before this commit: robot macaroni, 22 links, 21 joints
Joints:
- joint camera_joint: origin xyz=0.28 0 0.267 rpy=0 0.02 0 -> xyz=0.28 0 0.08 rpy=0 -0.04 0

Commit message: work in progress simple lane keeper

File: rr_description/urdf/sedani.urdf (robot description, URDF)
Before this commit: robot macaroni, 22 links, 21 joints
Joints:
- joint camera_joint: origin xyz=0.28 0 0.08 rpy=0 -0.04 0 -> xyz=0.28 0 0.09 rpy=0 -0.08 0

Commit message: initial setup for lane keeping test

File: rr_description/urdf/sedani.urdf (robot description, URDF)
Before this commit: robot macaroni, 22 links, 21 joints
Joints:
- joint base_footprint_to_chassis: origin xyz=0 0 0.036 rpy=0 0 0 -> xyz=0 0 0.079 rpy=0 0 0
- joint camera_joint: origin xyz=0.28 0 0.09 rpy=0 -0.08 0 -> xyz=0.28 0 0.18 rpy=0 -0.03 0

Commit message: changes from test day Feb 24

File: rr_description/urdf/sedani.urdf (robot description, URDF)
Before this commit: robot macaroni, 22 links, 21 joints
Joints:
- joint camera_joint: origin xyz=0.28 0 0.18 rpy=0 -0.03 0 -> xyz=0.28 0 0.1 rpy=0 -0.07 0
